Commit message: cleared model urdf

File: quadruped_robot/urdf/quadruped_robot.urdf (robot description, URDF)
Before this commit: robot quadruped_robot, 11 links, 10 joints
Links:
- removed link left_back_calf
- removed link left_back_foot
- removed link left_back_hip
- removed link left_back_leg
- removed link left_back_motor
- removed link left_forward_calf
- removed link left_forward_foot
- removed link left_forward_hip
- removed link left_forward_leg
- removed link left_forward_motor
Joints:
- removed joint body_left_back_motor
- removed joint body_left_forward_motor
- removed joint left_back_calf_foot
- removed joint left_back_hip_calf
- removed joint left_back_leg_hip
- removed joint left_back_motor_leg
- removed joint left_forward_calf_foot
- removed joint left_forward_hip_calf
- removed joint left_forward_leg_hip
- removed joint left_forward_motor_leg

Commit message: .

File: quadruped_robot/urdf/quadruped_robot.urdf (robot description, URDF)
Before this commit: robot quadruped_robot, 1 links, 0 joints
Links:
- added link world
Joints:
- added joint fixed: type fixed, parent world, child body

Commit message: added RPY track

File: quadruped_robot/urdf/quadruped_robot.urdf (robot description, URDF)
Before this commit: robot quadruped_robot, 2 links, 1 joints
Joints:
- removed joint fixed
- added joint world_body: type floating, parent world, child body, origin xyz=0 0 0.40 rpy=0 0 0

Commit message: updated URDF

File: quadruped_robot/urdf/quadruped_robot.urdf (robot description, URDF)
Before this commit: robot quadruped_robot, 2 links, 1 joints
Joints:
- joint world_body: origin xyz=0 0 0.40 rpy=0 0 0 -> xyz=0 0 0.5 rpy=0 0 0; type floating -> fixed

Commit message: fixed urdf

File: quadruped_robot/urdf/quadruped_robot.urdf (robot description, URDF)
Before this commit: robot quadruped_robot, 2 links, 1 joints
Links:
- removed link world
Joints:
- removed joint world_body

Commit message: .

File: quadruped_robot/urdf/quadruped_robot.urdf (robot description, URDF)
Before this commit: robot quadruped_robot, 1 links, 0 joints
Links:
- added link world
Joints:
- added joint world_body: type fixed, parent world, child body, origin xyz=0 0 0.5 rpy=0 0 0

Commit message: added damping and friction

File: quadruped_robot/urdf/quadruped_robot.urdf (robot description, URDF)
Before this commit: robot quadruped_robot, 2 links, 1 joints
Joints:
- joint world_body: type fixed -> floating

Commit message: .

File: quadruped_robot/urdf/quadruped_robot.urdf (robot description, URDF)
Before this commit: robot quadruped_robot, 2 links, 1 joints
Joints:
- joint world_body: origin xyz=0 0 0.5 rpy=0 0 0 -> xyz=0 0 0.45 rpy=0 0 0

Commit message: added plots

File: quadruped_robot/urdf/quadruped_robot.urdf (robot description, URDF)
Before this commit: robot quadruped_robot, 2 links, 1 joints
Joints:
- joint world_body: type floating -> fixed

Commit message: .

File: quadruped_robot/urdf/quadruped_robot.urdf (robot description, URDF)
Before this commit: robot quadruped_robot, 2 links, 1 joints
Links:
- removed link world
- link body: mass 0.614376972447432 -> 0.6
Joints:
- removed joint world_body

Commit message: fixed urdf and solved slipping problem in Gazebo

File: quadruped_robot/urdf/quadruped_robot.urdf (robot description, URDF)
Before this commit: robot quadruped_robot, 1 links, 0 joints
Links:
- removed link body
- added link imu_link, mass 0.001; collision box size=.001 .001 .001; visual box size=0.001 0.001 0.001
- added link trunk, mass 0.6; collision mesh filename=package://quadruped_robot/meshes/body.STL; visual mesh filename=package://quadruped_robot/meshes/body.STL
Joints:
- added joint imu_joint: type fixed, parent trunk, child imu_link, origin xyz=0 0 0 rpy=0 0 0
